File: eagle-files/controller-board.sch (EAGLE design)
At the start: 33 parts, among them CON1 to LEDs, CON3 AVR-ISP, CON4 to sliders, CON5 Snooze, CON6 RX/TX/gnd, CON6B Ser-GND, IC1 DS1307, IC2 ATMEGA328, X1 32.768kHz, X2 16MHz

Commit message: Add files via upload
Parts:
- R1: value 150Ω -> 2k2
Changed lines of the file:
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@@
 <setting verticaltext="up"/>
 </settings>
-<grid distance="0.05" unitdist="inch" unit="inch" style="lines" multiple="1" display="no" altdistance="0.01" altunitdist="inch" altunit="inch"/>
+<grid distance="0.1" unitdist="inch" unit="inch" style="lines" multiple="1" display="no" altdistance="0.01" altunitdist="inch" altunit="inch"/>
 <layers>
 <layer number="1" name="Top" color="4" fill="1" visible="no" active="no"/>
@@
 <part name="H3" library="holes" deviceset="MOUNT-HOLE" device="3.2" value="M3.2"/>
 <part name="LED1" library="led" deviceset="LED" device="3MM" value="green-3mm"/>
-<part name="R1" library="rcl" deviceset="R-EU_" device="0207/7" value="150Ω"/>
+<part name="R1" library="rcl" deviceset="R-EU_" device="0207/7" value="2k2"/>
 <part name="SUPPLY26" library="supply2" deviceset="+5V" device=""/>
 <part name="GND28" library="supply1" deviceset="GND" device=""/>
